File: Design/H00R5.sch (EAGLE design)
At the start: 1 part, among them P1 HEXABIT_17.32

Commit message: -Update the Schematic logo
Other:
- note added: "H00R5"
- note added: "H00R5_Frontend"
- note removed: "0"
- note removed: "H00R50"
- note removed: "H00R50_Frontend"
